Commit message: movo calibration

File: src/movo_calibration/results/calibrated_2019_02_12_16_31_04.urdf (robot description, URDF)
Before this commit: robot movo, 53 links, 52 joints
Joints:
- joint right_arm_half_joint: origin xyz=0.00000000 -0.20500000 0.00000000 rpy=-1.57079633 0.00000000 -0.01392410 -> xyz=0 -0.205 0 rpy=-1.570796325 0 0
- joint right_elbow_joint: origin xyz=0.00000000 0.00000000 -0.20500000 rpy=-1.57079633 0.00000000 0.03700006 -> xyz=0 0 -0.205 rpy=-1.570796325 0 0
- joint right_shoulder_lift_joint: origin xyz=0.00000000 0.00000000 -0.11875000 rpy=1.57079633 0.00000000 0.94894157 -> xyz=0 0 -0.11875 rpy=1.570796325 0 0
- joint right_shoulder_pan_joint: origin xyz=0.00000000 0.00000000 0.06250000 rpy=0.00000000 3.14159265 0.98853872 -> xyz=0 0 0.0625 rpy=0 3.14159265 0
